Commit message: measured weight implement

File: hexapod/resources/ASSY_phantom_urdf/urdf/ASSY_phantom_urdf(original).urdf (robot description, URDF)
Before this commit: robot ASSY_phantom_urdf, 20 links, 19 joints
Links:
- removed link reference_plate
- link LB_calf: mass 0.080679325949974 -> 0.0551626378910084
- link LB_foot: mass 0.103482656813031 -> 0.0652326466286265
- link LB_thigh: mass 0.0376750978794186 -> 0.0187184822855231
- link LF_calf: mass 0.0806793259499741 -> 0.0551626378910084
- link LF_foot: mass 0.103482656813031 -> 0.0652326466286266
- link LF_thigh: mass 0.0376750978794187 -> 0.0187184822855231
- link LM_calf: mass 0.0806793241220326 -> 0.055162636292801
- link LM_foot: mass 0.103482638943844 -> 0.0652326387878093
- link LM_thigh: mass 0.0376751009203242 -> 0.0187184853256138
- link RB_calf: mass 0.0806797008140726 -> 0.0551628381598268
- link RB_foot: mass 0.103482759622469 -> 0.0652327270508919
- link RB_thigh: mass 0.0376758208259914 -> 0.018718799941622
- link RF_calf: mass 0.0806797008140726 -> 0.0551628381598268
- link RF_foot: mass 0.10348275962247 -> 0.0652327270508921
- link RF_thigh: mass 0.0376758208259914 -> 0.0187187999416221
- link RM_calf: mass 0.0806797009667837 -> 0.0551628383199495
- link RM_foot: mass 0.103482743153361 -> 0.0652327208733654
- link RM_thigh: mass 0.0376758228348441 -> 0.0187188019506362
- link torso: mass 0.73121 -> 0.360578160137745
Joints:
- removed joint ref_to_torso_joint
- joint LB1: limit lower=-2.62 upper=2.62 effort=1.5 velocity=0 -> lower=-5.236 upper=5.236 effort=0 velocity=0
- joint LB2: limit lower=-2.62 upper=2.62 effort=1.5 velocity=0 -> lower=-5.236 upper=5.236 effort=0 velocity=0
- joint LB3: limit lower=-2.62 upper=2.62 effort=1.5 velocity=0 -> lower=-5.236 upper=5.236 effort=0 velocity=0
- joint LF1: limit lower=-2.62 upper=2.62 effort=1.5 velocity=0 -> lower=-5.236 upper=5.236 effort=0 velocity=0
- joint LF2: limit lower=-2.62 upper=2.62 effort=1.5 velocity=0 -> lower=-5.236 upper=5.236 effort=0 velocity=0
- joint LF3: limit lower=-2.62 upper=2.62 effort=1.5 velocity=0 -> lower=-5.236 upper=5.236 effort=0 velocity=0
- joint LM1: limit lower=-2.62 upper=2.62 effort=1.5 velocity=0 -> lower=-5.236 upper=5.236 effort=0 velocity=0
- joint LM2: limit lower=-2.62 upper=2.62 effort=1.5 velocity=0 -> lower=-5.236 upper=5.236 effort=0 velocity=0
- joint LM3: limit lower=-2.62 upper=2.62 effort=1.5 velocity=0 -> lower=-5.236 upper=5.236 effort=0 velocity=0
- joint RB1: limit lower=-2.62 upper=2.62 effort=1.5 velocity=0 -> lower=-5.236 upper=5.236 effort=0 velocity=0
- joint RB2: limit lower=-2.62 upper=2.62 effort=1.5 velocity=0 -> lower=-5.236 upper=5.236 effort=0 velocity=0
- joint RB3: limit lower=-2.62 upper=2.62 effort=1.5 velocity=0 -> lower=-5.236 upper=5.236 effort=0 velocity=0
- joint RF1: limit lower=-2.62 upper=2.62 effort=1.5 velocity=0 -> lower=-5.236 upper=5.236 effort=0 velocity=0
- joint RF2: limit lower=-2.62 upper=2.62 effort=1.5 velocity=0 -> lower=-5.236 upper=5.236 effort=0 velocity=0
- joint RF3: limit lower=-2.62 upper=2.62 effort=1.5 velocity=0 -> lower=-5.236 upper=5.236 effort=0 velocity=0
- joint RM1: limit lower=-2.62 upper=2.62 effort=1.5 velocity=0 -> lower=-5.236 upper=5.236 effort=0 velocity=0
- joint RM2: limit lower=-2.62 upper=2.62 effort=1.5 velocity=0 -> lower=-5.236 upper=5.236 effort=0 velocity=0
- joint RM3: limit lower=-2.62 upper=2.62 effort=1.5 velocity=0 -> lower=-5.236 upper=5.236 effort=0 velocity=0
