Commit message: added simple renderer, fixed hexapod legs, revised some render stuff

File: hexapod/resources/ASSY_phantom_urdf/urdf/ASSY_phantom_urdf.urdf (robot description, URDF)
Before this commit: robot ASSY_phantom_urdf, 20 links, 19 joints
Links:
- removed link reference_plate
Joints:
- removed joint ref_to_torso_joint
- joint LM1: origin xyz=0.1035 0 0 rpy=3.14159265358979 -1.5707963267949 0 -> xyz=0.1035 0 0 rpy=-1.5707963267949 -1.5707963267949 1.5707963267949 

Commit message: fixed robot reset mechanism

File: hexapod/resources/ASSY_phantom_urdf/urdf/ASSY_phantom_urdf.urdf (robot description, URDF)
Before this commit: robot ASSY_phantom_urdf, 19 links, 18 joints
Links:
- link LB_calf: mass 0.0551626378991534 -> 0.0551626378910084
- link LB_foot: mass 0.0659803620597775 -> 0.0652326466286265
- link LB_thigh: mass 0.0187184822855238 -> 0.0187184822855231
- link LF_calf: mass 0.0551626378991535 -> 0.0551626378910084
- link LF_foot: mass 0.0659803620597775 -> 0.0652326466286266
- link LF_thigh: mass 0.0187184822855238 -> 0.0187184822855231
- link LM_calf: mass 0.0551626363009457 -> 0.055162636292801
- link LM_foot: mass 0.0659803344728989 -> 0.0652326387878093
- link LM_thigh: mass 0.0187184853256144 -> 0.0187184853256138
- link RB_calf: mass 0.0551628381773647 -> 0.0551628381598268
- link RB_foot: mass 0.0659804422526083 -> 0.0652327270508919
- link RB_thigh: mass 0.0187187999416221 -> 0.018718799941622
- link RF_calf: mass 0.0551628381773646 -> 0.0551628381598268
- link RF_foot: mass 0.0659804422526083 -> 0.0652327270508921
- link RF_thigh: mass 0.018718799941622 -> 0.0187187999416221
- link RM_calf: mass 0.0551628383375633 -> 0.0551628383199495
- link RM_foot: mass 0.0659804165929113 -> 0.0652327208733654
- link torso: mass 0.361460112918338 -> 0.360578160137745
Joints:
- joint LB1: axis 0 1 0 -> 1 0 0; limit (none) -> lower=-5.236 upper=5.236 effort=0 velocity=0; origin xyz=0.0609100775541958 0 -0.121910077554196 rpy=0 -0.78539816339745 0 -> xyz=0.06091 0 -0.12191 rpy=0.7854 0 -1.5708; type continuous -> revolute
- joint LB2: axis 1 0 0 -> 0 0 1; limit (none) -> lower=-5.236 upper=5.236 effort=0 velocity=0; origin xyz=0 0.01844 -0.0519999999999999 rpy=-0.428439870509635 0 0 -> xyz=-0.01844 0 -0.052 rpy=1.5708 0.7854 0; type continuous -> revolute
- joint LB3: axis 1 0 0 -> 0 0 1; limit (none) -> lower=-5.236 upper=5.236 effort=0 velocity=0; origin xyz=0 0.0552704102679549 -0.0361826753434916 rpy=0.396828297419918 0 0 -> xyz=0.014589 -0.06443 0 rpy=0 0 1.3658; type continuous -> revolute
- joint LF1: axis 0 1 0 -> 1 0 0; limit (none) -> lower=-5.236 upper=5.236 effort=0 velocity=0; origin xyz=0.06091 0 0.12191 rpy=3.1416 -0.7854 -3.1416 -> xyz=0.06091 0 0.12191 rpy=2.3562 0 -1.5708; type continuous -> revolute
- joint LF2: axis 1 0 0 -> 0 0 1; limit (none) -> lower=-5.236 upper=5.236 effort=0 velocity=0; origin xyz=0 0.01844 -0.052 rpy=-0.428439870509635 0 0 -> xyz=-0.01844 0 -0.052 rpy=1.5708 0.7854 0; type continuous -> revolute
- joint LF3: axis 1 0 0 -> 0 0 1; limit (none) -> lower=-5.236 upper=5.236 effort=0 velocity=0; origin xyz=0 0.0552704102679548 -0.0361826753434916 rpy=0.396828297419917 0 0 -> xyz=0.014589 -0.06443 0 rpy=0 0 1.3658; type continuous -> revolute
- joint LM1: axis 0 1 0 -> 1 0 0; limit (none) -> lower=-5.236 upper=5.236 effort=0 velocity=0; origin xyz=0.1035 0 0 rpy=-1.5707963267949 -1.5707963267949 1.5707963267949  -> xyz=0.1035 0 0 rpy=1.5708 0 -1.5708; type continuous -> revolute
- joint LM2: axis 1 0 0 -> 0 0 1; limit (none) -> lower=-5.236 upper=5.236 effort=0 velocity=0; origin xyz=0 0.01844 -0.052 rpy=-0.428439870509635 0 0 -> xyz=-0.01844 0 -0.052 rpy=1.5708 0.7854 0; type continuous -> revolute
- joint LM3: axis 1 0 0 -> 0 0 1; limit (none) -> lower=-5.236 upper=5.236 effort=0 velocity=0; origin xyz=0 0.0552704102679549 -0.0361826753434916 rpy=0.396828297419917 0 0 -> xyz=0.014589 -0.06443 0 rpy=0 0 1.3658; type continuous -> revolute
- joint RB1: limit (none) -> lower=-5.236 upper=5.236 effort=0 velocity=0; origin xyz=-0.0609100775541957 0 -0.121910077554196 rpy=-2.35619449019234 0 1.5707963267949 -> xyz=-0.06091 0 -0.12191 rpy=2.3562 0 -1.5708; type continuous -> revolute
- joint RB2: axis 1 0 0 -> 0 0 1; limit (none) -> lower=-5.236 upper=5.236 effort=0 velocity=0; origin xyz=0.01844 0 0.052 rpy=0.428439870509635 0 -1.5707963267949 -> xyz=-0.01844 0 0.052 rpy=-1.5708 -0.7854 0; type continuous -> revolute
- joint RB3: axis 1 0 0 -> 0 0 1; limit (none) -> lower=-5.236 upper=5.236 effort=0 velocity=0; origin xyz=0 0.055270410267955 0.0361826753434918 rpy=-0.396828297419917 0 0 -> xyz=0.014589 -0.06443 0 rpy=0 0 1.3658; type continuous -> revolute
- joint RF1: limit (none) -> lower=-5.236 upper=5.236 effort=0 velocity=0; origin xyz=-0.0609100775541958 0 0.121910077554196 rpy=-0.785398163397452 0 1.5707963267949 -> xyz=-0.06091 0 0.12191 rpy=0.7854 0 -1.5708; type continuous -> revolute
- joint RF2: axis 1 0 0 -> 0 0 1; limit (none) -> lower=-5.236 upper=5.236 effort=0 velocity=0; origin xyz=0.0184400000000001 0 0.0520000000000002 rpy=0.428439870509634 0 -1.5707963267949 -> xyz=-0.01844 0 0.052 rpy=-1.5708 -0.7854 0; type continuous -> revolute
- joint RF3: axis 1 0 0 -> 0 0 1; limit (none) -> lower=-5.236 upper=5.236 effort=0 velocity=0; origin xyz=0 0.0627573500923168 0.0390014928378291 rpy=-0.396828297419917 0 0 -> xyz=0.014589 -0.06443 0 rpy=0 0 1.3658; type continuous -> revolute
- joint RM1: limit (none) -> lower=-5.236 upper=5.236 effort=0 velocity=0; origin xyz=-0.1035 0 0 rpy=-1.5707963267949 0 1.5707963267949 -> xyz=-0.1035 0 0 rpy=1.5708 0 -1.5708; type continuous -> revolute
- joint RM2: axis 1 0 0 -> 0 0 1; limit (none) -> lower=-5.236 upper=5.236 effort=0 velocity=0; origin xyz=0.0184400000000001 0 0.0520000000000001 rpy=0.428439870509635 0 -1.5707963267949 -> xyz=-0.01844 0 0.052 rpy=-1.5708 -0.7854 0; type continuous -> revolute
- joint RM3: axis 1 0 0 -> 0 0 1; limit (none) -> lower=-5.236 upper=5.236 effort=0 velocity=0; origin xyz=0 0.0552704102679548 0.0361826753434916 rpy=-0.396828297419917 0 0 -> xyz=0.014589 -0.06443 0 rpy=0 0 1.3658; type continuous -> revolute

Commit message: impl fixed torso

File: hexapod/resources/ASSY_phantom_urdf/urdf/ASSY_phantom_urdf.urdf (robot description, URDF)
Before this commit: robot ASSY_phantom_urdf, 20 links, 19 joints
Links:
- removed link reference_plate
Joints:
- removed joint ref_to_torso_joint

Commit message: hardware completed

File: hexapod/resources/ASSY_phantom_urdf/urdf/ASSY_phantom_urdf.urdf (robot description, URDF)
Before this commit: robot ASSY_phantom_urdf, 19 links, 18 joints
Links:
- link LB_calf: mass 0.080679325949974 -> 0.0806793209031789
- link LB_foot: mass 0.103482656813031 -> 0.103482657185437
- link LF_calf: mass 0.0806793259499741 -> 0.0806793209031788
- link LF_foot: mass 0.103482656813031 -> 0.103482657185437
- link LF_thigh: mass 0.0376750978794187 -> 0.0376750978794186
- link LM_calf: mass 0.0806793241220326 -> 0.0806793230410402
- link LM_foot: mass 0.103482638943844 -> 0.103482647116765
- link RB_calf: mass 0.0806797008140726 -> 0.0806796977247256
- link RB_foot: mass 0.103482759622469 -> 0.103482767086738
- link RF_calf: mass 0.0806797008140726 -> 0.0806796977247256
- link RF_foot: mass 0.10348275962247 -> 0.103482767086738
- link RM_calf: mass 0.0806797009667837 -> 0.0806796995241699
- link RM_foot: mass 0.103482743153361 -> 0.10348275106474
- link torso: mass 0.73121 -> 0.731212290700735
Joints:
- joint LB1: limit lower=-2.62 upper=2.62 effort=1.5 velocity=0 -> lower=-2.62 upper=2.62 effort=0 velocity=0; type revolute -> continuous
- joint LB2: limit lower=-2.62 upper=2.62 effort=1.5 velocity=0 -> lower=-2.62 upper=2.62 effort=0 velocity=0; origin xyz=-0.01844 0 -0.052 rpy=1.5708 0.7854 0 -> xyz=-0.01844 0 -0.052 rpy=1.5708 0 0; type revolute -> continuous
- joint LB3: limit lower=-2.62 upper=2.62 effort=1.5 velocity=0 -> lower=-2.62 upper=2.62 effort=0 velocity=0; origin xyz=0.014589 -0.06443 0 rpy=0 0 1.3658 -> xyz=0.014589 -0.06443 0 rpy=0 0 0.003125; type revolute -> continuous
- joint LF1: limit lower=-2.62 upper=2.62 effort=1.5 velocity=0 -> lower=-2.62 upper=2.62 effort=0 velocity=0; type revolute -> continuous
- joint LF2: limit lower=-2.62 upper=2.62 effort=1.5 velocity=0 -> lower=-2.62 upper=2.62 effort=0 velocity=0; origin xyz=-0.01844 0 -0.052 rpy=1.5708 0.7854 0 -> xyz=-0.01844 0 -0.052 rpy=1.5708 0 0; type revolute -> continuous
- joint LF3: limit lower=-2.62 upper=2.62 effort=1.5 velocity=0 -> lower=-2.62 upper=2.62 effort=0 velocity=0; origin xyz=0.014589 -0.06443 0 rpy=0 0 1.3658 -> xyz=0.014589 -0.06443 0 rpy=0 0 0.003125; type revolute -> continuous
- joint LM1: limit lower=-2.62 upper=2.62 effort=1.5 velocity=0 -> lower=-2.62 upper=2.62 effort=0 velocity=0; type revolute -> continuous
- joint LM2: limit lower=-2.62 upper=2.62 effort=1.5 velocity=0 -> lower=-2.62 upper=2.62 effort=0 velocity=0; origin xyz=-0.01844 0 -0.052 rpy=1.5708 0.7854 0 -> xyz=-0.01844 0 -0.052 rpy=1.5708 0 0; type revolute -> continuous
- joint LM3: limit lower=-2.62 upper=2.62 effort=1.5 velocity=0 -> lower=-2.62 upper=2.62 effort=0 velocity=0; origin xyz=0.014589 -0.06443 0 rpy=0 0 1.3658 -> xyz=0.014589 -0.06443 0 rpy=0 0 0.003125; type revolute -> continuous
- joint RB1: limit lower=-2.62 upper=2.62 effort=1.5 velocity=0 -> lower=-2.62 upper=2.62 effort=0 velocity=0; type revolute -> continuous
- joint RB2: limit lower=-2.62 upper=2.62 effort=1.5 velocity=0 -> lower=-2.62 upper=2.62 effort=0 velocity=0; origin xyz=-0.01844 0 0.052 rpy=-1.5708 -0.7854 0 -> xyz=-0.01844 0 0.052 rpy=-1.5708 0 0; type revolute -> continuous
- joint RB3: limit lower=-2.62 upper=2.62 effort=1.5 velocity=0 -> lower=-2.62 upper=2.62 effort=0 velocity=0; origin xyz=0.014589 -0.06443 0 rpy=0 0 1.3658 -> xyz=0.014589 -0.06443 0 rpy=0 0 0.003125; type revolute -> continuous
- joint RF1: limit lower=-2.62 upper=2.62 effort=1.5 velocity=0 -> lower=-2.62 upper=2.62 effort=0 velocity=0; type revolute -> continuous
- joint RF2: limit lower=-2.62 upper=2.62 effort=1.5 velocity=0 -> lower=-2.62 upper=2.62 effort=0 velocity=0; origin xyz=-0.01844 0 0.052 rpy=-1.5708 -0.7854 0 -> xyz=-0.01844 0 0.052 rpy=-1.5708 0 0; type revolute -> continuous
- joint RF3: limit lower=-2.62 upper=2.62 effort=1.5 velocity=0 -> lower=-2.62 upper=2.62 effort=0 velocity=0; origin xyz=0.014589 -0.06443 0 rpy=0 0 1.3658 -> xyz=0.014589 -0.06443 0 rpy=0 0 0.003125; type revolute -> continuous
- joint RM1: limit lower=-2.62 upper=2.62 effort=1.5 velocity=0 -> lower=-2.62 upper=2.62 effort=0 velocity=0; type revolute -> continuous
- joint RM2: limit lower=-2.62 upper=2.62 effort=1.5 velocity=0 -> lower=-2.62 upper=2.62 effort=0 velocity=0; origin xyz=-0.01844 0 0.052 rpy=-1.5708 -0.7854 0 -> xyz=-0.01844 0 0.052 rpy=-1.5708 0 0; type revolute -> continuous
- joint RM3: limit lower=-2.62 upper=2.62 effort=1.5 velocity=0 -> lower=-2.62 upper=2.62 effort=0 velocity=0; origin xyz=0.014589 -0.06443 0 rpy=0 0 1.3658 -> xyz=0.014589 -0.06443 0 rpy=0 0 0.003125; type revolute -> continuous
