Commit message: modified sampling

File: hexapod/resources/ASSY_phantom_urdf/urdf/old/ASSY_phantom_urdf.urdf (robot description, URDF)
Before this commit: robot ASSY_phantom_urdf, 19 links, 18 joints
Links:
- link LB_calf: mass 0.0806793209031789 -> 0.080679325949974
- link LB_foot: mass 0.103482657185437 -> 0.103482656813031
- link LF_calf: mass 0.0806793209031788 -> 0.0806793259499741
- link LF_foot: mass 0.103482657185437 -> 0.103482656813031
- link LF_thigh: mass 0.0376750978794186 -> 0.0376750978794187
- link LM_calf: mass 0.0806793230410402 -> 0.0806793241220326
- link LM_foot: mass 0.103482647116765 -> 0.103482638943844
- link RB_calf: mass 0.0806796977247256 -> 0.0806797008140726
- link RB_foot: mass 0.103482767086738 -> 0.103482759622469
- link RF_calf: mass 0.0806796977247256 -> 0.0806797008140726
- link RF_foot: mass 0.103482767086738 -> 0.10348275962247
- link RM_calf: mass 0.0806796995241699 -> 0.0806797009667837
- link RM_foot: mass 0.10348275106474 -> 0.103482743153361
- link torso: mass 0.731212290700735 -> 0.73121
Joints:
- joint LB1: limit lower=-2.62 upper=2.62 effort=0 velocity=0 -> lower=-2.62 upper=2.62 effort=1.5 velocity=0; type continuous -> revolute
- joint LB2: limit lower=-2.62 upper=2.62 effort=0 velocity=0 -> lower=-2.62 upper=2.62 effort=1.5 velocity=0; origin xyz=-0.01844 0 -0.052 rpy=1.5708 0 0 -> xyz=-0.01844 0 -0.052 rpy=1.5708 0.7854 0; type continuous -> revolute
- joint LB3: limit lower=-2.62 upper=2.62 effort=0 velocity=0 -> lower=-2.62 upper=2.62 effort=1.5 velocity=0; origin xyz=0.014589 -0.06443 0 rpy=0 0 0.003125 -> xyz=0.014589 -0.06443 0 rpy=0 0 1.3658; type continuous -> revolute
- joint LF1: limit lower=-2.62 upper=2.62 effort=0 velocity=0 -> lower=-2.62 upper=2.62 effort=1.5 velocity=0; type continuous -> revolute
- joint LF2: limit lower=-2.62 upper=2.62 effort=0 velocity=0 -> lower=-2.62 upper=2.62 effort=1.5 velocity=0; origin xyz=-0.01844 0 -0.052 rpy=1.5708 0 0 -> xyz=-0.01844 0 -0.052 rpy=1.5708 0.7854 0; type continuous -> revolute
- joint LF3: limit lower=-2.62 upper=2.62 effort=0 velocity=0 -> lower=-2.62 upper=2.62 effort=1.5 velocity=0; origin xyz=0.014589 -0.06443 0 rpy=0 0 0.003125 -> xyz=0.014589 -0.06443 0 rpy=0 0 1.3658; type continuous -> revolute
- joint LM1: limit lower=-2.62 upper=2.62 effort=0 velocity=0 -> lower=-2.62 upper=2.62 effort=1.5 velocity=0; type continuous -> revolute
- joint LM2: limit lower=-2.62 upper=2.62 effort=0 velocity=0 -> lower=-2.62 upper=2.62 effort=1.5 velocity=0; origin xyz=-0.01844 0 -0.052 rpy=1.5708 0 0 -> xyz=-0.01844 0 -0.052 rpy=1.5708 0.7854 0; type continuous -> revolute
- joint LM3: limit lower=-2.62 upper=2.62 effort=0 velocity=0 -> lower=-2.62 upper=2.62 effort=1.5 velocity=0; origin xyz=0.014589 -0.06443 0 rpy=0 0 0.003125 -> xyz=0.014589 -0.06443 0 rpy=0 0 1.3658; type continuous -> revolute
- joint RB1: limit lower=-2.62 upper=2.62 effort=0 velocity=0 -> lower=-2.62 upper=2.62 effort=1.5 velocity=0; type continuous -> revolute
- joint RB2: limit lower=-2.62 upper=2.62 effort=0 velocity=0 -> lower=-2.62 upper=2.62 effort=1.5 velocity=0; origin xyz=-0.01844 0 0.052 rpy=-1.5708 0 0 -> xyz=-0.01844 0 0.052 rpy=-1.5708 -0.7854 0; type continuous -> revolute
- joint RB3: limit lower=-2.62 upper=2.62 effort=0 velocity=0 -> lower=-2.62 upper=2.62 effort=1.5 velocity=0; origin xyz=0.014589 -0.06443 0 rpy=0 0 0.003125 -> xyz=0.014589 -0.06443 0 rpy=0 0 1.3658; type continuous -> revolute
- joint RF1: limit lower=-2.62 upper=2.62 effort=0 velocity=0 -> lower=-2.62 upper=2.62 effort=1.5 velocity=0; type continuous -> revolute
- joint RF2: limit lower=-2.62 upper=2.62 effort=0 velocity=0 -> lower=-2.62 upper=2.62 effort=1.5 velocity=0; origin xyz=-0.01844 0 0.052 rpy=-1.5708 0 0 -> xyz=-0.01844 0 0.052 rpy=-1.5708 -0.7854 0; type continuous -> revolute
- joint RF3: limit lower=-2.62 upper=2.62 effort=0 velocity=0 -> lower=-2.62 upper=2.62 effort=1.5 velocity=0; origin xyz=0.014589 -0.06443 0 rpy=0 0 0.003125 -> xyz=0.014589 -0.06443 0 rpy=0 0 1.3658; type continuous -> revolute
- joint RM1: limit lower=-2.62 upper=2.62 effort=0 velocity=0 -> lower=-2.62 upper=2.62 effort=1.5 velocity=0; type continuous -> revolute
- joint RM2: limit lower=-2.62 upper=2.62 effort=0 velocity=0 -> lower=-2.62 upper=2.62 effort=1.5 velocity=0; origin xyz=-0.01844 0 0.052 rpy=-1.5708 0 0 -> xyz=-0.01844 0 0.052 rpy=-1.5708 -0.7854 0; type continuous -> revolute
- joint RM3: limit lower=-2.62 upper=2.62 effort=0 velocity=0 -> lower=-2.62 upper=2.62 effort=1.5 velocity=0; origin xyz=0.014589 -0.06443 0 rpy=0 0 0.003125 -> xyz=0.014589 -0.06443 0 rpy=0 0 1.3658; type continuous -> revolute
