Commit message: hexapod-v2

File: hexapod/resources/ASSY_phantom_urdf/urdf/nocollision/ASSY_phantom_urdf.urdf (robot description, URDF)
Before this commit: robot ASSY_phantom_urdf, 19 links, 18 joints
Links:
- link LB_calf: geometry visual mesh filename=package://ASSY_phantom_urdf/meshes/LB_calf.STL
- link LB_thigh: geometry visual mesh filename=package://ASSY_phantom_urdf/meshes/LB_thigh.STL
- link LF_calf: geometry visual mesh filename=package://ASSY_phantom_urdf/meshes/LF_calf.STL
- link LF_thigh: geometry visual mesh filename=package://ASSY_phantom_urdf/meshes/LF_thigh.STL
- link LM_calf: geometry visual mesh filename=package://ASSY_phantom_urdf/meshes/LM_calf.STL
- link LM_thigh: geometry visual mesh filename=package://ASSY_phantom_urdf/meshes/LM_thigh.STL
- link RB_calf: geometry visual mesh filename=package://ASSY_phantom_urdf/meshes/RB_calf.STL
- link RB_thigh: geometry visual mesh filename=package://ASSY_phantom_urdf/meshes/RB_thigh.STL
- link RF_calf: geometry visual mesh filename=package://ASSY_phantom_urdf/meshes/RF_calf.STL
- link RF_thigh: geometry visual mesh filename=package://ASSY_phantom_urdf/meshes/RF_thigh.STL
- link RM_calf: geometry visual mesh filename=package://ASSY_phantom_urdf/meshes/RM_calf.STL
- link RM_thigh: geometry visual mesh filename=package://ASSY_phantom_urdf/meshes/RM_thigh.STL
- link torso: geometry visual mesh filename=package://ASSY_phantom_urdf/meshes/torso.STL
